File: NVG Monocular/NVG Monocular.kicad_pcb (KiCad board)
At the start: 2 copper layers, 23.5 x 28.6 mm, 32 parts, among them J1 I2C Breakout, J2 USB4105-GF-A, J3 breakout to header pin, J4 breakout to batt, U1 MP2696AGQ-0000-P

Commit message: V1.1 Corrected Header size to 2.54mm
Parts:
- J1, J3, J4, N1: footprint Connector_PinHeader_1.00mm:PinHeader_1x02_P1.00mm_Vertical -> Connector_PinSocket_2.54mm:PinSocket_1x02_P2.54mm_Vertical
- moved J3 9.76 mm to (158.5, 76.2)
- moved J1 6.51 mm to (158.5, 82.8)
- moved R4 4.69 mm to (155.1, 85.8), turned to 45 degrees
- moved R5 4.15 mm to (155.0, 88.1), turned to 45 degrees
- moved J4 3.28 mm to (158.5, 89.4)
- moved N1 0.41 mm to (158.5, 96.0)
Routing:
- net Net-(J3-Pin_1): track 14.0 -> 19.1 mm
- net Net-(U1-SDA): track 3.56 -> 8.20 mm
- net Net-(J3-Pin_2): track 10.3 -> 14.8 mm
- net Net-(U1-SCL): track 3.49 -> 6.86 mm
- net /SCL: track 6.79 -> 3.83 mm
- net /SDA: track 6.54 -> 3.83 mm
- net GND: track 2.72 -> 4.04 mm, vias 31 -> 23
Other:
- board text added: "MP2696A Breakout V1.1 Made with <3 by Siwen Long"
- board text removed: "MP2696A Breakout V1 Made with <3 by Siwen Long"
